Commit message: projects

File: catkin_ws/src/mrover/description/diff_rover/robot_core.xacro (robot description, xacro)
@@ -29,8 +29,8 @@
     <joint name="chassis_joint" type="fixed">
         <parent link="base_link"/>
-        <child link="chassis"/>
+        <child link="chassis_link"/>
         <origin xyz="-0.65 0 0"/>
     </joint>
-    <link name="chassis">
+    <link name="chassis_link">
         <visual>
             <origin xyz="0.65 0 0.415"/>
@@ -44,10 +44,10 @@
         </xacro:inertial_box>
     </link>
-    <gazebo reference="chassis">
+    <gazebo reference="chassis_link">
         <material>Gazebo/Orange</material>
     </gazebo>
     <!-- Back LEFT WHEEL LINK -->
     <joint name="back_left_wheel_joint" type="continuous">
-        <parent link="chassis"/>
+        <parent link="chassis_link"/>
         <child link="back_left_wheel"/>
         <origin xyz="0 0.525 0" rpy="-${pi/2} 0 0" />
@@ -75,5 +75,5 @@
     <!-- Back RIGHT WHEEL LINK -->
     <joint name="back_right_wheel_joint" type="continuous">
-        <parent link="chassis"/>
+        <parent link="chassis_link"/>
         <child link="back_right_wheel"/>
         <origin xyz="0 -0.525 0" rpy="${pi/2} 0 0" />
@@ -102,5 +102,5 @@
     <!-- Front LEFT WHEEL LINK -->
     <joint name="front_left_wheel_joint" type="continuous">
-        <parent link="chassis"/>
+        <parent link="chassis_link"/>
         <child link="front_left_wheel"/>
         <origin xyz="1.3 0.525 0" rpy="-${pi/2} 0 0" />
@@ -128,5 +128,5 @@
     <!-- RIGHT WHEEL LINK -->
     <joint name="front_right_wheel_joint" type="continuous">
-        <parent link="chassis"/>
+        <parent link="chassis_link"/>
         <child link="front_right_wheel"/>
         <origin xyz="1.3 -0.525 0" rpy="${pi/2} 0 0" />

File: catkin_ws/src/mrover/description/diff_rover/sensors/camera.xacro (robot description, xacro)
@@ -8,5 +8,5 @@
     <xacro:property name="far" value="8.0" />
     <joint name="camera_joint" type="fixed">
-        <parent link="chassis"/>
+        <parent link="chassis_link"/>
         <child link="camera_link"/>
         <origin xyz="1.315 0 0.70" rpy="0 0 0"/>

File: catkin_ws/src/mrover/description/diff_rover/sensors/lidar.xacro (robot description, xacro)
@@ -2,5 +2,5 @@
 <robot xmlns:xacro="http://www.ros.org/wiki/xacro" >
     <joint name="laser_joint" type="fixed">
-        <parent link="chassis"/>
+        <parent link="chassis_link"/>
         <child link="laser_frame"/>
         <origin xyz="1.0 0 0.83" rpy="0 0 0"/>

Commit message: add contoller

File: catkin_ws/src/mrover/description/diff_rover/robot_core.xacro (robot description, xacro)
@@ -2,4 +2,5 @@
 <robot xmlns:xacro="http://www.ros.org/wiki/xacro" >
     <xacro:include filename="inertial_macros.xacro"/>
+    <!-- <xacro:include filename="materials.xacro"/> -->
     <material name="white">
         <color rgba="1 1 1 1" />
@@ -29,8 +30,8 @@
     <joint name="chassis_joint" type="fixed">
         <parent link="base_link"/>
-        <child link="chassis"/>
+        <child link="chassis_link"/>
         <origin xyz="-0.65 0 0"/>
     </joint>
-    <link name="chassis">
+    <link name="chassis_link">
         <visual>
             <origin xyz="0.65 0 0.415"/>
@@ -44,10 +45,10 @@
         </xacro:inertial_box>
     </link>
-    <gazebo reference="chassis">
+    <gazebo reference="chassis_link">
         <material>Gazebo/Orange</material>
     </gazebo>
     <!-- Back LEFT WHEEL LINK -->
     <joint name="back_left_wheel_joint" type="continuous">
-        <parent link="chassis"/>
+        <parent link="chassis_link"/>
         <child link="back_left_wheel"/>
         <origin xyz="0 0.525 0" rpy="-${pi/2} 0 0" />
@@ -75,5 +76,5 @@
     <!-- Back RIGHT WHEEL LINK -->
     <joint name="back_right_wheel_joint" type="continuous">
-        <parent link="chassis"/>
+        <parent link="chassis_link"/>
         <child link="back_right_wheel"/>
         <origin xyz="0 -0.525 0" rpy="${pi/2} 0 0" />
@@ -102,5 +103,5 @@
     <!-- Front LEFT WHEEL LINK -->
     <joint name="front_left_wheel_joint" type="continuous">
-        <parent link="chassis"/>
+        <parent link="chassis_link"/>
         <child link="front_left_wheel"/>
         <origin xyz="1.3 0.525 0" rpy="-${pi/2} 0 0" />
@@ -128,5 +129,5 @@
     <!-- RIGHT WHEEL LINK -->
     <joint name="front_right_wheel_joint" type="continuous">
-        <parent link="chassis"/>
+        <parent link="chassis_link"/>
         <child link="front_right_wheel"/>
         <origin xyz="1.3 -0.525 0" rpy="${pi/2} 0 0" />

File: catkin_ws/src/mrover/description/diff_rover/sensors/lidar.xacro (robot description, xacro)
@@ -2,5 +2,5 @@
 <robot xmlns:xacro="http://www.ros.org/wiki/xacro" >
     <joint name="laser_joint" type="fixed">
-        <parent link="chassis"/>
+        <parent link="chassis_link"/>
         <child link="laser_frame"/>
         <origin xyz="1.0 0 0.83" rpy="0 0 0"/>

File: catkin_ws/src/mrover/description/steer_rover/robot_core.urdf.xacro (robot description, xacro)
@@ -5,4 +5,5 @@
     <xacro:include filename="sensors/lidar.xacro" />
     <xacro:include filename="sensors/camera.xacro" />
+    <!-- <xacro:include filename="gazebo/gazebo_control.xacro" /> -->
     <!-- <xacro:include filename="gazebo_control.xacro" />  -->
     <!-- <xacro:include filename="robot_core_ackermann.xacro" /> -->

File: catkin_ws/src/mrover/description/steer_rover/robot_core2.xacro (robot description, xacro)
@@ -16,4 +16,12 @@
     <!-- Base Link -->
     <link name="base_link" />
+    <!-- BASE_FOOTPRINT LINK -->
+    <joint name="base_footprint_joint" type="fixed">
+        <parent link="base_link"/>
+        <child link="base_footprint"/>
+        <origin xyz="0 0 0" rpy="0 0 0"/>
+    </joint>
+    <link name="base_footprint">
+    </link>
     <!-- Chassis -->
     <link name="chassis_link">
@@ -60,4 +68,18 @@
             <material name="invisible"/>
         </visual>
+        <collision>
+            <origin xyz="0 0 0" rpy="${PI/2} 0 ${PI/2}"/>
+            <geometry>
+                <cylinder length="0.01" radius="${wheel_radius}"/>
+            </geometry>
+        </collision>
+        <inertial>
+            <origin xyz="0 0 0" rpy="${PI/2} 0 ${PI/2}"/>
+            <mass value="${wheel_mass}"/>
+            <inertia
+                ixx="0.000270" ixy="0.0" ixz="0.0"
+                iyy="0.000270" iyz="0.0"
+                izz="0.000426"/>
+        </inertial>
     </link>
     <gazebo reference="virtual_rear_wheel">
@@ -154,4 +176,18 @@
         <material name="invisible"/>
         </visual>
+        <collision>
+                <origin xyz="0 0 0" rpy="${PI/2} 0 ${PI/2}"/>
+                <geometry>
+                    <cylinder length="0.01" radius="${wheel_radius}"/>
+                </geometry>
+        </collision>
+        <inertial>
+                <origin xyz="0 0 0" rpy="${PI/2} 0 ${PI/2}"/>
+                <mass value="${wheel_mass}"/>
+                <inertia
+                    ixx="0.000270" ixy="0.0" ixz="0.0"
+                    iyy="0.000270" iyz="0.0"
+                    izz="0.000426"/>
+        </inertial>
     </link>
     <gazebo reference="virtual_front_wheel">
@@ -200,5 +236,5 @@
         <limit lower="-0.4" upper="0.4" effort="100.0" velocity="0.0"/>
         <dynamics damping="0.2"/>
-        <mimic joint="virtual_front_wheel_joint" multiplier="1.0" offset="0.0"/>
+        <!-- <mimic joint="virtual_front_wheel_joint" multiplier="1.0" offset="0.0"/> -->
     </joint>
     <!-- front left steering -->
@@ -236,5 +272,5 @@
         <limit lower="-0.4" upper="0.4" effort="100.0" velocity="0.0"/>
         <dynamics damping="0.2"/>
-        <mimic joint="virtual_front_wheel_joint" multiplier="1.0" offset="0.0"/>
+        <!-- <mimic joint="virtual_front_wheel_joint" multiplier="1.0" offset="0.0"/> -->
     </joint>
 </robot>
