Commit message: update sim

File: catkin_ws/src/mrover/description/steer_rover/gazebo/gazebo_control.xacro (robot description, xacro)
@@ -3,10 +3,10 @@
   <gazebo>
     <plugin name="gazebo_ros_control" filename="libgazebo_ros_control.so">
-      <robotNamespace>/MYROBOT</robotNamespace>
-      <robotSimType>gazebo_ros_control/DefaultRobotHWSim</robotSimType>
+      <robotNamespace>/</robotNamespace>
+      <robotSimType>steer_bot_hardware_gazebo/SteerBotHardwareGazebo</robotSimType>
     </plugin>
   </gazebo>
 </robot>
-controller_manager:
+<!-- controller_manager:
   ros__parameters:
     update_rate: 50 # Hz
@@ -31,3 +31,3 @@
     pose_covariance_diagonal: [0.0, 7.0, 14.0, 21.0, 28.0, 35.0]
     position_feedback: false
-    use_stamped_vel: true
+    use_stamped_vel: true -->

File: catkin_ws/src/mrover/description/steer_rover/sensors/camera.xacro (robot description, xacro)
@@ -48,6 +48,13 @@
                 </clip>
             </camera>
-            <plugin name="camera_controller" filename="libgazebo_ros_camera.so">
+            <!-- <plugin name="camera_controller" filename="libgazebo_ros_camera.so">
                 <frame_name>camera_link_optical</frame_name>
+            </plugin> -->
+            <plugin name="gazebo_ros_camera" filename="libgazebo_ros_camera.so">
+                <robotNamespace>/</robotNamespace>
+                <cameraName>camera</cameraName>
+                <imageTopicName>image_raw</imageTopicName>
+                <cameraInfoTopicName>camera_info</cameraInfoTopicName>
+                <frameName>camera_link_optical</frameName>
             </plugin>
         </sensor>

File: catkin_ws/src/mrover/description/steer_rover/sensors/lidar.xacro (robot description, xacro)
@@ -15,5 +15,5 @@
                 <cylinder radius="${lidar_radius}" length="${lidar_length}"/>
             </geometry>
-            <material name="yellow"/>
+            <material name="blue"/>
         </visual>
         <collision>
@@ -27,13 +27,14 @@
     </link>
     <gazebo reference="laser_frame">
-        <material>Gazebo/Yellow</material>
-        <sensor name="laser" type="ray">
+        <material>Gazebo/Black</material>
+           <sensor name="laser" type="ray">
             <pose> 0 0 0 0 0 0 </pose>
             <visualize>false</visualize>
-            <update_rate>10</update_rate>
+            <update_rate>20</update_rate>
             <ray>
                 <scan>
                     <horizontal>
                         <samples>360</samples>
+                        <resolution>1</resolution>
                         <min_angle>-3.14</min_angle>
                         <max_angle>3.14</max_angle>
@@ -42,8 +43,19 @@
                 <range>
                     <min>0.3</min>
-                    <max>12</max>
+                    <max>12.0</max>
+                    <resolution>0.01</resolution>
                 </range>
+                <noise>
+                    <type>gaussian</type>
+                    <mean>0.0</mean>
+                    <stddev>0.01</stddev>
+                </noise>
             </ray>
-            <plugin name="laser_controller" filename="libgazebo_ros_ray_sensor.so">
+            <plugin name="gazebo_ros_laser_controller" filename="libgazebo_ros_laser.so">
+                <robotNamespace>/</robotNamespace>
+                <topicName>/scan</topicName>
+                <frameName>laser_frame</frameName>
+            </plugin>
+            <!-- <plugin name="laser_controller" filename="libgazebo_ros_ray_sensor.so">
                 <ros>
                     <argument>~/out:=scan</argument>
@@ -51,5 +63,5 @@
                 <output_type>sensor_msgs/LaserScan</output_type>
                 <frame_name>laser_frame</frame_name>
-            </plugin>
+            </plugin> -->
         </sensor>
     </gazebo>
