Commit message: update arduino

File: catkin_ws/src/mrover/description/diff_rover/gazebo/gazebo_control_diff.xacro (robot description, xacro)
@@ -1,7 +1,35 @@
 <?xml version="1.0"?>
 <robot xmlns:xacro="http://www.ros.org/wiki/xacro">
+    <xacro:property name="wheel_radius" value="0.1397" />
+    <xacro:property name="wheel_separation" value="1.05" />
     <gazebo>
-        <plugin name="diff_drive" filename="libgazebo_ros_diff_drive.so">
-            <numWheelPairs>2</numWheelPairs>
+        <plugin name="diff_drive" filename="libgazebo_ros_diff_drive.so">>
+            <ros>
+                <namespace>/</namespace>
+                <remapping>cmd_vel:=cmd_vel</remapping>
+                <remapping>odom:=odom</remapping>
+            </ros>
+            <robotNamespace/>
+            <alwaysOn>true</alwaysOn>
+	        <updateRate>100</updateRate>
+            <!-- <controlFrequency>50</controlFrequency> -->
+            <wheelSeparation>${wheel_separation}</wheelSeparation>
+            <wheelDiameter>${2*wheel_radius}</wheelDiameter>
+            <wheelAcceleration>0.0</wheelAcceleration>
+            <wheelTorque>5.0</wheelTorque>
+            <odometryTopic>odom</odometryTopic>
+	        <odometryFrame>odom</odometryFrame>
+            <baseFrame>chassis</baseFrame>
+            <!-- <leftJoint>front_left_wheel_joint</leftJoint> -->
+            <leftJoint>rear_left_wheel_joint</leftJoint>
+            <!-- <rightJoint>front_right_wheel_joint</rightJoint> -->
+            <rightJoint>rear_right_wheel_joint</rightJoint>
+            <robotBaseFrame>base_link</robotBaseFrame>
+            <publishWheelTF>true</publishWheelTF>
+            <publishOdom>true</publishOdom>
+            <publishWheelJointState>true</publishWheelJointState>
+            <legacyMode>false</legacyMode>
+        </plugin>
+            <!-- <numWheelPairs>2</numWheelPairs>
             <alwaysOn>true</alwaysOn>
             <updateRate>20</updateRate>
@@ -9,7 +37,7 @@
             <rightJoint>rear_right_wheel_joint</rightJoint>
             <leftJoint>front_left_wheel_joint</leftJoint>
-            <rightJoint>front_right_wheel_joint</rightJoint>
+            <rightJoint>front_right_wheel_joint</rightJoint> -->
             <!-- kinematics -->
-            <wheelSeparation>1.05</wheelSeparation>
+            <!-- <wheelSeparation>1.05</wheelSeparation>
             <wheelSeparation>1.05</wheelSeparation>
             <wheelDiameter>0.2794</wheelDiameter>
@@ -22,28 +50,28 @@
             <publishTf>1</publishTf>
             <publishWheelJointState>true</publishWheelJointState>
-            <robotBaseFrame>base_link</robotBaseFrame>
+            <robotBaseFrame>base_link</robotBaseFrame> -->
             <!-- Number of wheel pairs -->
-            <num_wheel_pairs>2</num_wheel_pairs>
+            <!-- <num_wheel_pairs>2</num_wheel_pairs> -->
             <!-- back Wheel Information -->
-            <left_joint>rear_left_wheel_joint</left_joint>
-            <right_joint>rear_right_wheel_joint</right_joint>
+            <!-- <left_joint>rear_left_wheel_joint</left_joint>
+            <right_joint>rear_right_wheel_joint</right_joint> -->
             <!-- front Wheel Information -->
-            <left_joint>front_left_wheel_joint</left_joint>
-            <right_joint>front_right_wheel_joint</right_joint>
+            <!-- <left_joint>front_left_wheel_joint</left_joint>
+            <right_joint>front_right_wheel_joint</right_joint> -->
             <!-- kinematics -->
-            <wheel_separation>1.05</wheel_separation>
+            <!-- <wheel_separation>1.05</wheel_separation>
             <wheel_separation>1.05</wheel_separation>
             <wheel_diameter>0.2794</wheel_diameter>
-            <wheel_diameter>0.2794</wheel_diameter>
+            <wheel_diameter>0.2794</wheel_diameter> -->
             <!-- Limits -->
-            <max_wheel_torque>200</max_wheel_torque>
-            <max_wheel_acceleration>20.0</max_wheel_acceleration>
+            <!-- <max_wheel_torque>200</max_wheel_torque>
+            <max_wheel_acceleration>20.0</max_wheel_acceleration> -->
             <!-- Output -->
-            <odometry_frame>odom_demo</odometry_frame>
+            <!-- <odometry_frame>odom_demo</odometry_frame>
             <robot_base_frame>base_link</robot_base_frame>
             <publish_odom>true</publish_odom>
             <publish_odom_tf>true</publish_odom_tf>
-            <publish_wheel_tf>true</publish_wheel_tf>
-        </plugin>
+            <publish_wheel_tf>true</publish_wheel_tf> -->
+        <!-- </plugin> -->
     </gazebo>
 </robot>

File: catkin_ws/src/mrover/description/diff_rover/robot.urdf.xacro (robot description, xacro)
@@ -4,8 +4,8 @@
     <xacro:include filename="sensors/lidar.xacro" />
     <xacro:include filename="sensors/camera.xacro" />
+    <xacro:include filename="gazebo/gazebo_control_diff.xacro" />
     <!-- <xacro:include filename="sensors/camera.xacro" /> -->
     <!-- <xacro:include filename="gazwbo_control_steer.xacro" />
     <xacro:include filename="lidar.xacro" /> -->
-    <!-- <xacro:include filename="gazebo_control.xacro" />  -->
     <!-- <xacro:include filename="robot_core_ackermann.xacro" /> -->
     <!-- <xacro:include filename="mrover_ackermann.xacro" />

File: catkin_ws/src/mrover/description/diff_rover/sensors/camera.xacro (robot description, xacro)
@@ -44,6 +44,13 @@
                 </clip>
             </camera>
-            <plugin name="camera_controller" filename="libgazebo_ros_camera.so">
+            <!-- <plugin name="camera_controller" filename="libgazebo_ros_camera.so">
                 <frame_name>camera_link_optical</frame_name>
+            </plugin> -->
+            <plugin name="gazebo_ros_camera" filename="libgazebo_ros_camera.so">
+                <robotNamespace>/</robotNamespace>
+                <cameraName>camera</cameraName>
+                <imageTopicName>image_raw</imageTopicName>
+                <cameraInfoTopicName>camera_info</cameraInfoTopicName>
+                <frameName>camera_link_optical</frameName>
             </plugin>
         </sensor>

File: catkin_ws/src/mrover/description/steer_bot_description/urdf/steer_bot.urdf.xacro (robot description, xacro)
@@ -1,9 +1,4 @@
 <?xml version="1.0"?>
 <!--
-  Robot model adapted from https://github.com/CIR-KIT/steer_drive_ros/blob/kinetic-devel/steer_drive_controller/test/common/urdf/steerbot.xacro
-  Modifications:
-    Remove base_footprint link. Useful for navigation but not necessary for a simple example.
-    Added materials for URDF
-    Updated inertials
   Geometry:
     The Ackermann steering controllers require the longitudinal
@@ -18,5 +13,4 @@
   <xacro:include filename="wheel.xacro"/>
   <xacro:include filename="inertial_macros.xacro"/>
-    <!-- <xacro:include filename="materials.xacro"/> -->
   <xacro:property name="robot_namespace" value="/steer_bot"/>
   <!-- Gazebo plugins -->
@@ -41,5 +35,5 @@
   <xacro:property name="wheel_radius" value="0.1397" />
   <xacro:property name="wheel_thickness" value="0.125" />
-  <xacro:property name="wheel_mass" value="1" />
+  <xacro:property name="wheel_mass" value="8" />
   <!-- Steering link dimensions -->
   <xacro:property name="steer_radius" value="0.05" />
@@ -76,4 +70,10 @@
         <box size="${base_length} ${base_width} ${base_height}"/>
       </geometry>
+      <contact>
+        <ode>
+          <mu>20</mu>
+          <mu2>20</mu2>
+        </ode>
+      </contact>
     </collision>
     <xacro:solid_cuboid_inertial

File: catkin_ws/src/mrover/description/steer_bot_description/urdf/wheel.xacro (robot description, xacro)
@@ -1,5 +1,4 @@
 <?xml version="1.0"?>
 <!--
-  Robot model adapted from https://github.com/CIR-KIT/steer_drive_ros/blob/kinetic-devel/steer_drive_controller/test/common/urdf/wheel.xacro
   Modifications:
     <transmissions> elements have been updated and added to 'front_steer'.
@@ -98,4 +97,10 @@
           <cylinder radius="${steer_radius}" length="${steer_thickness}"/>
         </geometry>
+        <contact>
+          <ode>
+            <mu>20</mu>
+            <mu2>20</mu2>
+          </ode>
+        </contact>
       </collision>
       <xacro:solid_cylinder_inertial
@@ -126,4 +131,10 @@
           <cylinder radius="${wheel_radius}" length="${wheel_thickness}"/>
         </geometry>
+        <contact>
+          <ode>
+            <mu>20</mu>
+            <mu2>20</mu2>
+          </ode>
+        </contact>
       </collision>
       <xacro:solid_cylinder_inertial
@@ -187,4 +198,10 @@
           <cylinder radius="${wheel_radius}" length="${wheel_thickness}"/>
         </geometry>
+        <contact>
+          <ode>
+            <mu>20</mu>
+            <mu2>20</mu2>
+          </ode>
+        </contact>
       </collision>
       <xacro:solid_cylinder_inertial
@@ -235,4 +252,10 @@
           <cylinder radius="${wheel_radius}" length="${wheel_thickness}"/>
         </geometry>
+        <contact>
+          <ode>
+            <mu>20</mu>
+            <mu2>20</mu2>
+          </ode>
+        </contact>
       </collision>
       <xacro:solid_cylinder_inertial
@@ -276,4 +299,10 @@
           <cylinder radius="${wheel_radius}" length="${wheel_thickness}"/>
         </geometry>
+        <contact>
+          <ode>
+            <mu>20</mu>
+            <mu2>20</mu2>
+          </ode>
+        </contact>
       </collision>
       <xacro:solid_cylinder_inertial
